File: _schematics/v3.brd (EAGLE design)
At the start: 40 x 37.5 mm, 25 parts, among them J1 AC_IN, J2 IR_LED, J3 IO0, Q1 N-MOSFET-SOT23, Q2 N-MOSFET-SOT23, U1 ESP-12F, U2 LD117ASTR

Commit message: Update schematics
Parts:
- R1, R6, R7, R8: device resistor:R0805 -> resistor:R0603
- moved R6 1.71 mm to (6.99, 30.5), turned to 0 degrees
- moved R8 1.16 mm to (28.9, 24.0), turned to 90 degrees
- moved R4 0.48 mm to (31.4, 25.6)
- moved R7 0.35 mm to (7.94, 28.1)
Connections:
- net N$7 renamed EN
Routing:
- net 3V3: track 73.9 -> 74.9 mm
- net GND: track 28.8 -> 29.2 mm, vias 9 -> 10
- added copper zone on layer 1, net GND
Other:
- outline, holes or cut-outs redrawn
- board text added: "IR Remote"
- board text added: "by RouNdeL"
- board text added: "git.io/vhU1T"
- board text added: "© 2018 Krzysztof Zdulski"
